File: KiCad/PT100_Datalogger/Connectors.kicad_sch (KiCad schematic)
At the start: 23 parts, among them J1 PWR, J13 HLK-LD2410C, J3 Screw_Terminal_01x02, J7 CT_SW

Commit message: Finished KiCad PCB REV A
Parts:
- removed D10, D6: ESD5Z12T1G, Diode_SMD:D_SOD-523, symbol Device:D_TVS
- removed D36: ESD5Z3V3, Diode_SMD:D_SOD-523, symbol Diode:ESD5Zxx
- removed H1: MountingHole_Pad, MountingHole:MountingHole_3.2mm_M3, symbol Mechanical:MountingHole
- removed J13: HLK-LD2410C, Connector_Molex:Molex_KK-254_AE-6410-05A_1x05_P2.54mm_Vertical, symbol Connector_Generic:Conn_01x05
- removed J7: CT_SW, Connector_Molex:Molex_KK-254_AE-6410-02A_1x02_P2.54mm_Vertical, symbol Connector_Generic:Conn_01x02
- added C6: DE1B3RA471KN4AP01F, Capacitor_THT:C_Disc_D7.5mm_W5.0mm_P10.00mm, symbol Device:C
- added D11, D8, D9: ESD5Z12T1G, Diode_SMD:D_SOD-523, symbol Device:D_Zener
- added H1: MountingHole_Pad, MountingHole:MountingHole_3.2mm_M3_Pad, symbol Mechanical:MountingHole_Pad
- added J14: PWR, Connector_JST:JST_VH_B3P-VH_1x03_P3.96mm_Vertical, symbol Connector_Generic:Conn_01x03
- added J2: Conn_01x04, Connector_Molex:Molex_KK-254_AE-6410-04A_1x04_P2.54mm_Vertical, symbol Connector_Generic:Conn_01x04
- added J6: RTD, Connector_Molex:Molex_KK-254_AE-6410-05A_1x05_P2.54mm_Vertical, symbol Connector_Generic:Conn_01x05
- added J7: MAX7219, Connector_Molex:Molex_KK-254_AE-6410-05A_1x05_P2.54mm_Vertical, symbol Connector_Generic:Conn_01x05
- added U2: SN74LVC245APW, Package_SO:TSSOP-20_4.4x6.5mm_P0.65mm, symbol Logic_LevelTranslator:SN74LVC245APW
- J3: value Screw_Terminal_01x02 -> TC
Connections:
- net CT is gone; now on net +5V: C16.1
- net +5V: now also J2.4 (Pin_4), J7.1 (Pin_1), U2.1 (DIR), U2.20 (VCC)
- net GND: now also J3.3 (Pin_3), C6.2, D11.2 (A), D8.2 (A), D9.2 (A), H1.1, J2.3 (Pin_3), J6.1 (Pin_1), J7.2 (Pin_2), U2.10 (GND), U2.5 (A4), U2.6 (A5), U2.7 (A6), U2.8 (A7), U2.9 (A8); no longer H3.1, J3.1 (Pin_1)
- net at D13.1 (K), R52.1, R56.1: now also J3.1 (Pin_1); no longer J3.3 (Pin_3)
- net U1RX renamed U0TXD
- net U0TXD: now also J2.1 (Pin_1)
- net U1TX renamed U0RXD
- net U0RXD: now also J2.2 (Pin_2)
- new net: D11.1 (K), J7.3 (Pin_3), U2.18 (B1)
- new net: D9.1 (K), J7.4 (Pin_4), U2.17 (B2)
- new net: D8.1 (K), J7.5 (Pin_5), U2.16 (B3)
- new net D_CS: U2.3 (A2)
- new net Earth_Clean: C6.1, J14.3 (Pin_3)
- new net L1: J14.2 (Pin_2)
- new net LEVEL_OE: U2.19 (~{OE})
- new net MOSI: U2.2 (A1)
- new net NEUT: J14.1 (Pin_1)
- new net RTD_FN: J6.2 (Pin_2)
- new net RTD_FP: J6.5 (Pin_5)
- new net RTD_INN: J6.3 (Pin_3)
- new net RTD_INP: J6.4 (Pin_4)
- new net SCK: U2.4 (A3)
- no-connect marks 0 -> 6
Other:
- moved on the sheet: D7, J1, J3
