File: KiCad/PT100_Datalogger/Power.kicad_sch (KiCad schematic)
At the start: 12 parts, among them J14 691406710003B, U4 LDL212PV33R

Commit message: Finished KiCad PCB REV A
Parts:
- removed J14: 691406710003B, Personal:691406710003B, symbol Connector:Screw_Terminal_01x03
- D21, D4: footprint LED_THT:LED_D5.0mm -> LED_SMD:LED_0603_1608Metric_Pad1.05x0.95mm_HandSolder
Other:
- note added: "Keep ground isolated"
