File: KiCad/PT100_Datalogger/USB.kicad_sch (KiCad schematic)
At the start: 17 parts, among them J2 USB_C_Receptacle, Q16 MMBT3904, Q17 MMBT3904, U2 CP2102N-Axx-xQFN28

Commit message: Finished KiCad PCB REV A
Parts:
- removed C6, C7: 10uF, Capacitor_SMD:C_0805_2012Metric_Pad1.18x1.45mm_HandSolder, symbol Device:C
- removed D11, D12, D8: TSD05CDYFR, Diode_SMD:D_SOD-323_HandSoldering, symbol Device:D_TVS
- removed D9: B5819W, Diode_SMD:D_SOD-123, symbol Device:D_Schottky
- removed J2: USB_C_Receptacle, Personal:CONN_CU3216SASBLR004-NH_CVI, symbol Connector:USB_C_Receptacle_USB2.0_14P
- removed Q16, Q17: MMBT3904, Package_TO_SOT_SMD:SOT-23_Handsoldering, symbol Transistor_BJT:Q_NPN_BEC
- removed R17, R18: 5k1, Resistor_SMD:R_0603_1608Metric_Pad0.98x0.95mm_HandSolder, symbol Device:R
- removed R2: 1K, Resistor_SMD:R_0603_1608Metric_Pad0.98x0.95mm_HandSolder, symbol Device:R
- removed R3: 22K1, Resistor_SMD:R_0603_1608Metric_Pad0.98x0.95mm_HandSolder, symbol Device:R
- removed R4: 47K5, Resistor_SMD:R_0603_1608Metric_Pad0.98x0.95mm_HandSolder, symbol Device:R
- removed R5, R6: 10K, Resistor_SMD:R_0603_1608Metric_Pad0.98x0.95mm_HandSolder, symbol Device:R
- removed U2: CP2102N-Axx-xQFN28, Package_DFN_QFN:QFN-28-1EP_5x5mm_P0.5mm_EP3.35x3.35mm, symbol Interface_USB:CP2102N-Axx-xQFN28
- added D14, D2, D3: TSD05CDYFR, Diode_SMD:D_SOD-323_HandSoldering, symbol Device:D_TVS
- added D5: B5819W, Diode_SMD:D_SOD-123, symbol Device:D_Schottky
- added J5: CU3216SASBLR004-NH, Personal:CONN_CU3216SASBLR004-NH_CVI, symbol Connector:USB_C_Receptacle_USB2.0_14P
- added R23, R24: 5k1, Resistor_SMD:R_0603_1608Metric_Pad0.98x0.95mm_HandSolder, symbol Device:R
Connections:
- net +5V: now also D5.1 (K)
- net GND: now also D14.1 (A1), D2.1 (A1), D3.1 (A1), J5.A1 (GND), J5.A12 (GND), J5.B1 (GND), J5.B12 (GND), J5.S1 (SHIELD), R23.2, R24.2
- net USB_D+: now also D14.2 (A2), J5.A6 (D+), J5.B6 (D+)
- net USB_D-: now also D2.2 (A2), J5.A7 (D-), J5.B7 (D-)
- net VBUS: now also D3.2 (A2), D5.2 (A), J5.A4 (VBUS), J5.A9 (VBUS), J5.B4 (VBUS), J5.B9 (VBUS)
- new net: J5.A5 (CC1), R23.1
- new net: J5.B5 (CC2), R24.1
- no-connect marks 16 -> 0
